File: schematic_312503_eagle.sch (EAGLE design)
At the start: 0 parts

Commit message: Update schematic_312503_eagle.sch
Replaced empty Eagle schematics export with a working copy.
Parts:
- added C1, C4: 470µF 25V LS 5mm, common:CAP_POLARIZED
- added C10: 2.2nF, common:FILM_CAPACITOR
- added C11: 0.47µF film 100V, common:CAP
- added C12: 0.1µF, common:CAP
- added C13: 2.2nF, common:CAP
- added C14, C8, C9: 22µF 25V LS 3/5mm, common:CAP_POLARIZED
- added C2: 0.1µF 310Vac 10% 15mm, common:X2_CAP
- added C3, C6: 2200pF 250VAC 15mm, common:Y2_CAP
- added C5: 4700µF 25V LS 10mm, common:CAP_POLARIZED
- added C7: 4700µF 16V, common:CAP_POLARIZED
- added D1: 1N4148F, common:1N4148F
- added D2: 1N4148F_1, common:1N4148F_1
- added D3, D5: 1N5401, common:1N5401
- added D4, D9: 1N4001, common:1N4001
- added D6: 1N5822, common:1N5822
- added D7: 5v6 ZENER, common:DEV_D7
- added F1: 315mA 250V, common:FUSE
- added L1: ?? uH, common:IND_MAGN_CORE1
- added Q1: D45H2, common:PNP
- added R1, R2: 182 ohm 1%, common:RES
- added R10, R11, R12, R3: 47 ohm, common:RES
- added R4: 1.5kohm, common:RES
- added R5: 4.7kohm, common:RES
- added R6: 100kohm 10%, common:RES
- added R7: 47kohm 1%, common:RES
- added R8: 1.5kohm 1%, common:RES
- added R9: 12kohm 1%, common:RES
- added T1: 18/36V, common:ISMET
- added THY2: C106D, common:SCR_4A_400V
- added U1: L7912CV, common:L7912CV
- added U2: L7812CV, common:L7812CV
- added U3: SG3524BN, common:SG3524BN
Connections:
- new net +12V: C9.PLUS, D2.A, U2.OUT
- new net +5V: C14.PLUS, C7.MINUS, D9.A, L1.2, R11.2, R12.1, R5.1, U3.I_LIM_+
- new net -12V: C8.MINUS, D1.K, U1.OUT
- new net GND: C1.PLUS, C11.1, C12.2, C13.1, C14.MINUS, C4.MINUS, C5.MINUS, C7.PLUS, C8.PLUS, C9.MINUS, D6.A, R10.1, R4.2, R8.1, R9.2, T1.0, THY2.K, U1.GND, U2.GND, U3.EMIT_1, U3.EMIT_2, U3.GND, U3.SHUTDN
- new net Main: C10.1, C4.PLUS, C5.PLUS, D2.C, D3.K, D5.K, Q1.E, R3.2, U2.IN, U3.VCC
- new net Net_0: C2.1, C3.2, F1.1
- new net Net_1: C3.1, C6.1
- new net Net_10: R1.2, R2.2, U3.COL_1, U3.COL_2
- new net Net_12: D6.K, L1.1, Q1.C
- new net Net_15: R4.1, R5.2, U3.IN_-
- new net Net_16: R6.2, U3.COMP
- new net Net_17: C11.2, R6.1
- new net Net_19: C12.1, R7.1, R8.2, U3.IN_+
- new net Net_2: D5.A, T1.18_AC@2
- new net Net_20: R9.1, U3.RT
- new net Net_21: C13.2, U3.CT
- new net Net_22: D7.K, R11.1
- new net Net_24: C2.2, C6.2, T1.AC@2
- new net Net_25: C10.2, Q1.B, R1.1, R2.1, R3.1
- new net Net_3: F1.2, T1.AC@1
- new net Net_4: D3.A, D4.C, T1.18_AC@1
- new net Net_5: D7.A, R10.2, THY2.G
- new net Net_6: C1.MINUS, D1.A, D4.A, U1.IN
- new net Net_7: R7.2, U3.REF_OUT
- new net Net_8: D9.C, R12.2, THY2.A, U3.I_LIM_-
Other:
- note added: "#"
- note added: "+12V"
- note added: "+12V Regulator"
- note added: "+5V"
- note added: "-12V"
- note added: "-12V Regulator"
- note added: "0.1µF"
- note added: "0.1µF 310Vac 10% 15mm"
- note added: "0.1µF 310Vac 10% LS 15mm"
- note added: "0.1µF LS 5mm"
- note added: "0.47µF film 100V"
- note added: "0.47µF film 100V LS 5mm"
- note added: "1"
- note added: "1.5kohm"
- note added: "1.5kohm 1%"
- note added: "10"
- note added: "100kohm 10%"
- note added: "10A06-T, 10A02, 1N5552 etc."
- note added: "11"
- note added: "12"
- note added: "12kohm 1%"
- note added: "13"
- note added: "14"
- note added: "15"
- note added: "16"
- note added: "17"
- note added: "18"
- note added: "18/36V"
- note added: "182 ohm 1%"
- note added: "19"
- note added: "1N4001"
- note added: "1N4148F"
- note added: "1N5401"
- note added: "1N5822"
- note added: "2"
- note added: "2.2nF"
- note added: "2.2nF LS 5mm"
- note added: "20"
- note added: "21"
- note added: "22"
- note added: "2200pF 250VAC 15mm"
- note added: "2200pF LS 15mm"
- note added: "22µF 25V LS 3/5mm"
- note added: "23"
- note added: "24"
- note added: "25"
- note added: "26"
- note added: "27"
- note added: "28"
- note added: "29"
- note added: "3"
- note added: "3.0V (33mA) between COL and Q1 base"
- note added: "30"
- note added: "31"
- note added: "315mA 250V"
- note added: "32"
- note added: "33"
- note added: "34"
- note added: "35"
- note added: "36"
- note added: "37"
- note added: "38"
- note added: "39"
- note added: "4"
- note added: "4.7kohm"
- note added: "40"
- note added: "41"
- note added: "42"
- note added: "47 ohm"
- note added: "4700µF 16V"
- note added: "4700µF 25V LS 10mm"
- note added: "470µF 25V LS 5mm"
- note added: "47kohm 1%"
- note added: "5"
- note added: "5V switching supply circuit"
- note added: "5v6 ZENER"
- note added: "6"
- note added: "7"
- note added: "8"
- note added: "9"
- note added: "?? uH"
- note added: "?? µH"
- note added: "A500 waiting disk to be inserted, after warmup:"
- note added: "B81123C1222M289, MPRY2W1220FC00MSSD"
- note added: "C1"
- note added: "C10"
- note added: "C106D"
- note added: "C106DG/C106D1G (4A) SJ6008VS2TP (8A)"
- note added: "C11"
- note added: "C12"
- note added: "C13"
- note added: "C13+R9 = 50kHz"
- note added: "C14"
- note added: "C2"
- note added: "C3"
- note added: "C4"
- note added: "C5"
- note added: "C6"
- note added: "C7"
- note added: "C8"
- note added: "C9"
- note added: "CAP"
- note added: "CAP_POLARIZED"
- note added: "CMF60182R00FHEK"
- note added: "COL"
- note added: "D1"
- note added: "D2"
- note added: "D3"
- note added: "D4"
- note added: "D45H11, D45H8 etc."
- note added: "D45H2"
- note added: "D5"
- note added: "D6"
- note added: "D7"
- note added: "D9"
- note added: "EARTH"
- note added: "EEUFR1C472"
- note added: "EEUFR1E471YB"
- note added: "ELBK350ELL472ALN3S"
- note added: "F1"
- note added: "F17724102000"
- note added: "FUSE"
- note added: "Film capacitor"
- note added: "GND"
- note added: "IND_MAGN_CORE1"
- note added: "IN_+, IN_-: 1.2V"
- note added: "ISMET"
- note added: "L"
- note added: "L1"
- note added: "L7812CV"
- note added: "L7912CV"
- note added: "LIM-"
- note added: "May be replaced with"
- note added: "N"
- note added: "Name"
- note added: "PNP"
- note added: "Q1"
- note added: "Q1 base: 14.8µs off (2V), 5.2µs on (21V), 26% duty"
- note added: "R1"
- note added: "R10"
- note added: "R11"
- note added: "R12"
- note added: "R2"
- note added: "R3"
- note added: "R4"
- note added: "R5"
- note added: "R6"
- note added: "R7"
- note added: "R8"
- note added: "R9"
- note added: "RES"
- note added: "RefDes"
- note added: "SCR 4A 400V"
- note added: "SG3524BN"
- note added: "T1"
- note added: "THY2"
- note added: "U1"
- note added: "U2"
- note added: "U3"
- note added: "UC2524AN"
- note added: "VCC"
- note added: "Value"
- note added: "Vcc abt. 21V"
- note added: "WCAP-PT5H 870235673001"
- note added: "X2 CAP"
- note added: "Y2 CAP"
- note added: "crowbar"
- note added: "feedback"
